Commit message: Materiales asignados para piezas del brazo robotico

File: resultados/Robot_URDF/assembly.SLDASM/urdf/assembly.SLDASM.urdf (robot description, URDF)
Before this commit: robot assembly.SLDASM, 5 links, 4 joints
Links:
- link base_link: mass 20.049 -> 156.38
- link link_1: mass 14.514675782209 -> 39.19
- link link_2: mass 15.4604615363391 -> 41.743
- link link_3: mass 12.0600722432213 -> 32.562
- link link_4: mass 1.1764892790594 -> 2.1294
Joints:
- joint joint_2: origin xyz=0 -0.16 0 rpy=-1.5708 0 0 -> xyz=0 -0.160000000000001 0 rpy=-1.5707963267949 0 0
