Commit message: correccion de nombre del archivo

File: resultados/Robot_URDF/assembly_sldsam/urdf/assembly_sldsam.urdf (robot description, URDF)
Before this commit: robot assembly.SLDASM, 5 links, 4 joints
Links:
- link base_link: mass 156.38 -> 156.384128910965; geometry collision mesh filename=package://assembly_sldsam/meshes/base_link.STL; visual mesh filename=package://assembly_sldsam/meshes/base_link.STL
- link link_1: mass 39.19 -> 39.1896246119642; geometry collision mesh filename=package://assembly_sldsam/meshes/link_1.STL; visual mesh filename=package://assembly_sldsam/meshes/link_1.STL
- link link_2: mass 41.743 -> 41.7432461481157; geometry collision mesh filename=package://assembly_sldsam/meshes/link_2.STL; visual mesh filename=package://assembly_sldsam/meshes/link_2.STL
- link link_3: mass 32.562 -> 32.5621950566976; geometry collision mesh filename=package://assembly_sldsam/meshes/link_3.STL; visual mesh filename=package://assembly_sldsam/meshes/link_3.STL
- link link_4: mass 2.1294 -> 2.12944559509751; geometry collision mesh filename=package://assembly_sldsam/meshes/link_4.STL; visual mesh filename=package://assembly_sldsam/meshes/link_4.STL
Joints:
- joint joint_1: origin xyz=0 0 0.16 rpy=1.5708 0 0 -> xyz=0 0 0.160000000000001 rpy=1.5707963267949 0 0
