Commit message: urdf corregido

File: resultados/Robot_URDF/assembly/urdf/assembly.urdf (robot description, URDF)
Before this commit: robot assembly_sldsam, 5 links, 4 joints
Links:
- link base_link: geometry collision mesh filename=package://assembly/meshes/base_link.STL; visual mesh filename=package://assembly/meshes/base_link.STL
- link link_1: geometry collision mesh filename=package://assembly/meshes/link_1.STL; visual mesh filename=package://assembly/meshes/link_1.STL
- link link_2: geometry collision mesh filename=package://assembly/meshes/link_2.STL; visual mesh filename=package://assembly/meshes/link_2.STL
- link link_3: geometry collision mesh filename=package://assembly/meshes/link_3.STL; visual mesh filename=package://assembly/meshes/link_3.STL
- link link_4: geometry collision mesh filename=package://assembly/meshes/link_4.STL; visual mesh filename=package://assembly/meshes/link_4.STL

Commit message: correccion de robot final

File: resultados/Robot_URDF/assembly/urdf/assembly.urdf (robot description, URDF)
Before this commit: robot assembly, 5 links, 4 joints
Links:
- link base_link: mass 156.38 -> 156.384128910965
Joints:
- joint joint_2: origin xyz=0 0 0.496 rpy=-1.5708 0 0 -> xyz=0 0 0.496 rpy=1.5708 0 0
- joint joint_3: origin xyz=0 -0.5 0 rpy=-3.1416 0 0 -> xyz=0 0.5 0 rpy=-3.1416 0 1.8978
- joint joint_4: origin xyz=-0.41805 0.17024 0 rpy=0 0 3.1416 -> xyz=0.145 -0.42746 0 rpy=3.1416 0 -1.2438

Commit message: correccion

File: resultados/Robot_URDF/assembly/urdf/assembly.urdf (robot description, URDF)
Before this commit: robot assembly, 5 links, 4 joints
Links:
- link link_1: mass 39.19 -> 39.1896246119642
- link link_2: mass 41.743 -> 41.7432461481157
- link link_3: mass 32.562 -> 32.5621952947336
