Commit message: assembly prueba 2

File: src/assembly/urdf/assembly.urdf (robot description, URDF)
Before this commit: robot assembly, 5 links, 4 joints
Links:
- added link world
- link link_3: mass 32.5621950566976 -> 32.5621952947336
- link link_4: mass 2.12944559509751 -> 2.1294
Joints:
- added joint base_joint: type fixed, parent world, child base_link, origin xyz=0.0 0.0 0.17 rpy=0 0 0
- joint joint_1: axis 0 1 0 -> 0 0 1; limit lower=0 upper=3.142 effort=300 velocity=3 -> lower=-3.142 upper=3.142 effort=300 velocity=3; origin xyz=0 0 0.160000000000001 rpy=1.5707963267949 0 0 -> xyz=0 0 0 rpy=0 0 0
- joint joint_2: axis 0 -1 0 -> 0 0 1; origin xyz=0 -0.160000000000001 0 rpy=-1.5707963267949 0 0 -> xyz=0 0 0.496 rpy=1.5708 0 0
- joint joint_3: axis 0 -1 0 -> 0 0 1; limit lower=0 upper=3.142 effort=200 velocity=3 -> lower=-3.142 upper=0 effort=200 velocity=3; origin xyz=0 0 0 rpy=0 0 0 -> xyz=0 0.5 0 rpy=-3.1416 0 1.8978
- joint joint_4: axis 0 1 0 -> 0 0 1; limit lower=0 upper=-3.142 effort=200 velocity=3 -> lower=-3.142 upper=0 effort=200 velocity=3; origin xyz=0 0 0 rpy=0 0 0 -> xyz=0.145 -0.42746 0 rpy=3.1416 0 -1.2438

Commit message: EL robot no colisiona prueba 1

File: src/assembly/urdf/assembly.urdf (robot description, URDF)
Before this commit: robot assembly, 6 links, 5 joints
Joints:
- joint joint_3: origin xyz=0 0.5 0 rpy=-3.1416 0 1.8978 -> xyz=0 0.5 0 rpy=0 0 0

Commit message: robot movimiento 1

File: src/assembly/urdf/assembly.urdf (robot description, URDF)
Before this commit: robot assembly, 6 links, 5 joints
Joints:
- joint joint_3: origin xyz=0 0.5 0 rpy=0 0 0 -> xyz=0 0.5 0 rpy=-3.1416 0 1.8978

Commit message: Se volvio a exportar el movit_robot_soldador_sim

File: src/assembly/urdf/assembly.urdf (robot description, URDF)
Before this commit: robot assembly, 6 links, 5 joints
Joints:
- joint joint_3: limit lower=-3.142 upper=0 effort=200 velocity=3 -> lower=0 upper=3.142 effort=200 velocity=3

File: src/moveit_robot_soldador_sim/config/gazebo_assembly.urdf (robot description, URDF)
Before this commit: robot assembly, 6 links, 5 joints
Joints:
- joint joint_3: limit lower=-3.142 upper=0 effort=200 velocity=3 -> lower=0 upper=3.142 effort=200 velocity=3
